File: pcb/pcb.kicad_sch (KiCad schematic)
At the start: 32 parts, among them SW1 EVQ-P7J01P, SW2 EVQ-P7J01P, U1 SN74AHCT1G125DBVR, U2 XIAO-RP2350-DIP, U3 TMAG5273A2QDBVR, U4 TMAG5273B2QDBVR, U5 TMAG5273C2QDBVR

Commit message: BOM correction
Parts:
- U3: value TMAG5273A2QDBVR -> TMAG5273A1QDBVR; symbol space_mouse:TMAG5273A2QDBVR -> space_mouse:TMAG5273A1QDBVR
- U4: value TMAG5273B2QDBVR -> TMAG5273B1QDBVR; symbol space_mouse:TMAG5273A2QDBVR -> space_mouse:TMAG5273A1QDBVR
- U5: value TMAG5273C2QDBVR -> TMAG5273C1QDBVR; symbol space_mouse:TMAG5273A2QDBVR -> space_mouse:TMAG5273A1QDBVR
Changed lines of the file:
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@@
 	)
 	(symbol
-		(lib_id "space_mouse:TMAG5273A2QDBVR")
+		(lib_id "space_mouse:TMAG5273A1QDBVR")
 		(at 199.39 109.22 0)
 		(unit 1)
@@
 			)
 		)
-		(property "Value" "TMAG5273C2QDBVR"
+		(property "Value" "TMAG5273C1QDBVR"
 			(at 215.9 101.6 0)
 			(show_name no)
@@
 	)
 	(symbol
-		(lib_id "space_mouse:TMAG5273A2QDBVR")
+		(lib_id "space_mouse:TMAG5273A1QDBVR")
 		(at 109.22 109.22 0)
 		(unit 1)
@@
 			)
 		)
-		(property "Value" "TMAG5273A2QDBVR"
+		(property "Value" "TMAG5273A1QDBVR"
 			(at 125.73 101.6 0)
 			(show_name no)
@@
 	)
 	(symbol
-		(lib_id "space_mouse:TMAG5273A2QDBVR")
+		(lib_id "space_mouse:TMAG5273A1QDBVR")
 		(at 154.94 109.22 0)
 		(unit 1)
@@
 			)
 		)
-		(property "Value" "TMAG5273B2QDBVR"
+		(property "Value" "TMAG5273B1QDBVR"
 			(at 171.45 101.6 0)
 			(show_name no)
